File: SPS-BellDriver.sch (KiCad schematic (older format))
At the start: 61 parts, among them IC1 TSR_1-2433, J1 Jack-DC, J2 Screw_Terminal_01x02, J3 Screw_Terminal_01x02, J4 Screw_Terminal_01x02, J5 Screw_Terminal_01x05, J6 Screw_Terminal_01x02, J7 Screw_Terminal_01x02, J8 Screw_Terminal_01x05, J9 Screw_Terminal_01x02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

Commit message: updates
Parts:
- added H1: 1590B, SamacSys_Parts:1590B, symbol SamacSys_Parts:1590B
- D10, D11, D12, D13, D14, D9: footprint Diode_THT:D_DO-41_SOD81_P3.81mm_Vertical_KathodeUp -> Diode_THT:D_DO-41_SOD81_P7.62mm_Horizontal
- R24: footprint Resistor_THT:R_Axial_DIN0207_L6.3mm_D2.5mm_P2.54mm_Vertical -> Resistor_THT:R_Axial_DIN0207_L6.3mm_D2.5mm_P5.08mm_Vertical
